Commit message: trying to spawn 2 robots

File: myrobot_description/robots/myrobot.urdf.xacro (robot description, xacro)
@@ -5,4 +5,4 @@
   	<xacro:arg name="gazebo" value="${gazebo}"/>
   </xacro:include>
-  <xacro:myrobot connected_to='world'/>
+  <xacro:myrobot connected_to='world' arm_id='myrobot'/>
 </robot>

File: myrobot_description/robots/myrobot.xacro (robot description, xacro)
@@ -1,5 +1,5 @@
 <?xml version="1.0" encoding="utf-8"?>
 <robot xmlns:xacro="http://www.ros.org/wiki/xacro" name="myrobot">
-<xacro:macro name="myrobot" params="arm_id:='myrobot' package_name:='myrobot_description' connected_to:='' xyz:='0 0 0' rpy:='0 0 0' hardware_interface:=''">
+  <xacro:macro name="myrobot" params="arm_id:='myrobot' package_name:='myrobot_description' connected_to:='' xyz:='0 0 0' rpy:='0 0 0' hardware_interface:=''">
     <xacro:unless value="${not connected_to}">
       <link name="${connected_to}"/>
@@ -10,163 +10,179 @@
       </joint>
     </xacro:unless>
+    <xacro:property name="PI" value="3.1415926535897931"/>
+    <xacro:property name="mass" value="1" />
+    <!-- arbitrary value for mass -->
+    <xacro:property name="width" value="0.1" />
+    <!-- Square dimensions (widthxwidth) of beams -->
+    <xacro:property name="height1" value="2" />
+    <!-- Link 1 -->
+    <xacro:property name="height2" value="1" />
+    <!-- Link 2 -->
+    <xacro:property name="height3" value="1" />
+    <!-- Link 3 -->
+    <!-- Base Link -->
+    <link name="${arm_id}_link1">
+      <collision>
+        <origin xyz="0 0 0" rpy="0 0 0"/>
+        <geometry>
+          <mesh filename="package://myrobot_description/meshes/Base.stl"/>
+        </geometry>
+      </collision>
+      <visual>
+        <origin xyz="0 0 0" rpy="0 0 0"/>
+        <geometry>
+          <mesh filename="package://myrobot_description/meshes/Base.stl"/>
+        </geometry>
+        <material name="">
+          <color rgba="1 1 1 1"/>
+        </material>
+      </visual>
+      <inertial>
+        <origin xyz="0 0 0" rpy="0 0 0"/>
+        <mass value="${mass}"/>
+        <inertia ixx="${mass / 12.0 * (width*width + height1*height1)}" ixy="0.0" ixz="0.0" iyy="${mass / 12.0 * (height1*height1 + width*width)}" iyz="0.0" izz="${mass / 12.0 * (width*width + width*width)}"/>
+      </inertial>
+    </link>
+    <joint name="${arm_id}_joint1" type="continuous">
+      <parent link="${arm_id}_link1"/>
+      <child link="${arm_id}_link2"/>
+      <origin xyz="0 0 0.07" rpy="0 0 0"/>
+      <axis xyz="0 0 1"/>
+      <dynamics damping="0.7"/>
+    </joint>
+    <!-- Middle Link -->
+    <link name="${arm_id}_link2">
+      <collision>
+        <origin xyz="0 0 0" rpy="0 0 0"/>
+        <geometry>
+          <mesh filename="package://myrobot_description/meshes/Link1.stl"/>
+        </geometry>
+      </collision>
+      <visual>
+        <origin xyz="0 0 0" rpy="0 0 0"/>
+        <geometry>
+          <mesh filename="package://myrobot_description/meshes/Link1.stl"/>
+        </geometry>
+        <material name="">
+          <color rgba="1 1 1 1"/>
+        </material>
+      </visual>
+      <inertial>
+        <origin xyz="0 0 0" rpy="0 0 0"/>
+        <mass value="${mass}"/>
+        <inertia ixx="${mass / 12.0 * (width*width + height2*height2)}" ixy="0.0" ixz="0.0" iyy="${mass / 12.0 * (height2*height2 + width*width)}" iyz="0.0" izz="${mass / 12.0 * (width*width + width*width)}"/>
+      </inertial>
+    </link>
+    <joint name="${arm_id}_joint2" type="continuous">
+      <parent link="${arm_id}_link2"/>
+      <child link="${arm_id}_link3"/>
+      <origin xyz="0.08 0 0.12" rpy="${pi/2} 0 ${pi/2}"/>
+      <axis xyz="0 0 1"/>
+      <dynamics damping="0.7"/>
+    </joint>
+    <!-- Top Link -->
+    <link name="${arm_id}_link3">
+      <collision>
+        <origin xyz="0 0 0" rpy="0 0 0"/>
+        <geometry>
+          <mesh filename="package://myrobot_description/meshes/Link2.stl"/>
+        </geometry>
+      </collision>
+      <visual>
+        <origin xyz="0 0 0" rpy="0 0 0"/>
+        <geometry>
+          <mesh filename="package://myrobot_description/meshes/Link2.stl"/>
+        </geometry>
+        <material name="">
+          <color rgba="1 1 1 1"/>
+        </material>
+      </visual>
+      <inertial>
+        <origin xyz="0 0 0" rpy="0 0 0"/>
+        <mass value="${mass}"/>
+        <inertia ixx="${mass / 12.0 * (width*width + height3*height3)}" ixy="0.0" ixz="0.0" iyy="${mass / 12.0 * (height3*height3 + width*width)}" iyz="0.0" izz="${mass / 12.0 * (width*width + width*width)}"/>
+      </inertial>
+    </link>
+    <joint name="${arm_id}_joint3" type="continuous">
+      <parent link="${arm_id}_link3"/>
+      <child link="${arm_id}_link4"/>
+      <origin xyz="0 0.43 0" rpy="0 0 0"/>
+      <axis xyz="0 0 1"/>
+      <dynamics damping="0.7"/>
+    </joint>
+    <!-- Top Link -->
+    <link name="${arm_id}_link4">
+      <collision>
+        <origin xyz="0 0 0" rpy="0 0 0"/>
+        <geometry>
+          <mesh filename="package://myrobot_description/meshes/Link3.stl"/>
+        </geometry>
+      </collision>
+      <visual>
+        <origin xyz="0 0 0" rpy="0 0 0"/>
+        <geometry>
+          <mesh filename="package://myrobot_description/meshes/Link3.stl"/>
+        </geometry>
+        <material name="">
+          <color rgba="1 1 1 1"/>
+        </material>
+      </visual>
+      <inertial>
+        <origin xyz="0 0 0" rpy="0 0 0"/>
+        <mass value="${mass}"/>
+        <inertia ixx="${mass / 12.0 * (width*width + height3*height3)}" ixy="0.0" ixz="0.0" iyy="${mass / 12.0 * (height3*height3 + width*width)}" iyz="0.0" izz="${mass / 12.0 * (width*width + width*width)}"/>
+      </inertial>
+    </link>
+    <!-- GAZEBO -->
     <xacro:arg name="gazebo" default="true"/>
     <xacro:arg name="hardware_interface" default="EffortJointInterface"/>
-    <xacro:if value="$(arg gazebo)">
-      <xacro:include filename="$(find myrobot_description)/robots/myrobot.gazebo.xacro"/>
-    </xacro:if>
-  <xacro:property name="PI" value="3.1415926535897931"/>
-  <xacro:property name="mass" value="1" />
-  <!-- arbitrary value for mass -->
-  <xacro:property name="width" value="0.1" />
-  <!-- Square dimensions (widthxwidth) of beams -->
-  <xacro:property name="height1" value="2" />
-  <!-- Link 1 -->
-  <xacro:property name="height2" value="1" />
-  <!-- Link 2 -->
-  <xacro:property name="height3" value="1" />
-  <!-- Link 3 -->
-  <!-- Base Link -->
-  <link name="${arm_id}_link1">
-    <collision>
-      <origin xyz="0 0 0" rpy="0 0 0"/>
-      <geometry>
-        <mesh filename="package://myrobot_description/meshes/Base.stl"/>
-      </geometry>
-    </collision>
-    <visual>
-      <origin xyz="0 0 0" rpy="0 0 0"/>
-      <geometry>
-        <mesh filename="package://myrobot_description/meshes/Base.stl"/>
-      </geometry>
-      <material name="">
-        <color rgba="1 1 1 1"/>
-      </material>
-    </visual>
-    <inertial>
-      <origin xyz="0 0 0" rpy="0 0 0"/>
-      <mass value="${mass}"/>
-      <inertia ixx="${mass / 12.0 * (width*width + height1*height1)}" ixy="0.0" ixz="0.0" iyy="${mass / 12.0 * (height1*height1 + width*width)}" iyz="0.0" izz="${mass / 12.0 * (width*width + width*width)}"/>
-    </inertial>
-  </link>
-  <joint name="${arm_id}_joint1" type="continuous">
-    <parent link="${arm_id}_link1"/>
-    <child link="${arm_id}_link2"/>
-    <origin xyz="0 0 0.07" rpy="0 0 0"/>
-    <axis xyz="0 0 1"/>
-    <dynamics damping="0.7"/>
-  </joint>
-  <!-- Middle Link -->
-  <link name="${arm_id}_link2">
-    <collision>
-      <origin xyz="0 0 0" rpy="0 0 0"/>
-      <geometry>
-        <mesh filename="package://myrobot_description/meshes/Link1.stl"/>
-      </geometry>
-    </collision>
-    <visual>
-      <origin xyz="0 0 0" rpy="0 0 0"/>
-      <geometry>
-        <mesh filename="package://myrobot_description/meshes/Link1.stl"/>
-      </geometry>
-      <material name="">
-        <color rgba="1 1 1 1"/>
-      </material>
-    </visual>
-    <inertial>
-      <origin xyz="0 0 0" rpy="0 0 0"/>
-      <mass value="${mass}"/>
-      <inertia ixx="${mass / 12.0 * (width*width + height2*height2)}" ixy="0.0" ixz="0.0" iyy="${mass / 12.0 * (height2*height2 + width*width)}" iyz="0.0" izz="${mass / 12.0 * (width*width + width*width)}"/>
-    </inertial>
-  </link>
-  <joint name="${arm_id}_joint2" type="continuous">
-    <parent link="${arm_id}_link2"/>
-    <child link="${arm_id}_link3"/>
-    <origin xyz="0.08 0 0.12" rpy="${pi/2} 0 ${pi/2}"/>
-    <axis xyz="0 0 1"/>
-    <dynamics damping="0.7"/>
-  </joint>
-  <!-- Top Link -->
-  <link name="${arm_id}_link3">
-    <collision>
-      <origin xyz="0 0 0" rpy="0 0 0"/>
-      <geometry>
-        <mesh filename="package://myrobot_description/meshes/Link2.stl"/>
-      </geometry>
-    </collision>
-    <visual>
-      <origin xyz="0 0 0" rpy="0 0 0"/>
-      <geometry>
-        <mesh filename="package://myrobot_description/meshes/Link2.stl"/>
-      </geometry>
-      <material name="">
-        <color rgba="1 1 1 1"/>
-      </material>
-    </visual>
-    <inertial>
-      <origin xyz="0 0 0" rpy="0 0 0"/>
-      <mass value="${mass}"/>
-      <inertia ixx="${mass / 12.0 * (width*width + height3*height3)}" ixy="0.0" ixz="0.0" iyy="${mass / 12.0 * (height3*height3 + width*width)}" iyz="0.0" izz="${mass / 12.0 * (width*width + width*width)}"/>
-    </inertial>
-  </link>
-  <joint name="${arm_id}_joint3" type="continuous">
-    <parent link="${arm_id}_link3"/>
-    <child link="${arm_id}_link4"/>
-    <origin xyz="0 0.43 0" rpy="0 0 0"/>
-    <axis xyz="0 0 1"/>
-    <dynamics damping="0.7"/>
-  </joint>
-  <!-- Top Link -->
-  <link name="${arm_id}_link4">
-    <collision>
-      <origin xyz="0 0 0" rpy="0 0 0"/>
-      <geometry>
-        <mesh filename="package://myrobot_description/meshes/Link3.stl"/>
-      </geometry>
-    </collision>
-    <visual>
-      <origin xyz="0 0 0" rpy="0 0 0"/>
-      <geometry>
-        <mesh filename="package://myrobot_description/meshes/Link3.stl"/>
-      </geometry>
-      <material name="">
-        <color rgba="1 1 1 1"/>
-      </material>
-    </visual>
-    <inertial>
-      <origin xyz="0 0 0" rpy="0 0 0"/>
-      <mass value="${mass}"/>
-      <inertia ixx="${mass / 12.0 * (width*width + height3*height3)}" ixy="0.0" ixz="0.0" iyy="${mass / 12.0 * (height3*height3 + width*width)}" iyz="0.0" izz="${mass / 12.0 * (width*width + width*width)}"/>
-    </inertial>
-  </link>
-  <transmission name="${arm_id}_joint1_trans">
-    <type>transmission_interface/SimpleTransmission</type>
-    <joint name="${arm_id}_joint1">
-      <hardwareInterface>hardware_interface/EffortJointInterface</hardwareInterface>
-    </joint>
-    <actuator name="${arm_id}_joint1_motor">
-      <hardwareInterface>hardware_interface/EffortJointInterface</hardwareInterface>
-      <mechanicalReduction>1</mechanicalReduction>
-    </actuator>
-  </transmission>
-  <transmission name="${arm_id}_joint2_trans">
-    <type>transmission_interface/SimpleTransmission</type>
-    <joint name="${arm_id}_joint2">
-      <hardwareInterface>hardware_interface/EffortJointInterface</hardwareInterface>
-    </joint>
-    <actuator name="${arm_id}_joint2_motor">
-      <hardwareInterface>hardware_interface/EffortJointInterface</hardwareInterface>
-      <mechanicalReduction>1</mechanicalReduction>
-    </actuator>
-  </transmission>
-  <transmission name="${arm_id}_joint3_trans">
-    <type>transmission_interface/SimpleTransmission</type>
-    <joint name="${arm_id}_joint3">
-      <hardwareInterface>hardware_interface/EffortJointInterface</hardwareInterface>
-    </joint>
-    <actuator name="${arm_id}_joint3_motor">
-      <hardwareInterface>hardware_interface/EffortJointInterface</hardwareInterface>
-      <mechanicalReduction>1</mechanicalReduction>
-    </actuator>
-  </transmission>
-</xacro:macro>
+    <gazebo>
+      <plugin name="gazebo_ros_control" filename="libgazebo_ros_control.so">
+        <!-- <robotNamespace>/</robotNamespace> -->
+        <robotNamespace>${arm_id}</robotNamespace>
+      </plugin>
+    </gazebo>
+    <gazebo reference="${arm_id}_link1">
+      <turnGravityOff>false</turnGravityOff>
+    </gazebo>
+    <gazebo reference="${arm_id}_link2">
+      <turnGravityOff>false</turnGravityOff>
+    </gazebo>
+    <gazebo reference="${arm_id}_link3">
+      <turnGravityOff>false</turnGravityOff>
+    </gazebo>
+    <gazebo reference="${arm_id}_link4">
+      <turnGravityOff>false</turnGravityOff>
+    </gazebo>
+    <transmission name="${arm_id}_joint1_trans">
+      <type>transmission_interface/SimpleTransmission</type>
+      <joint name="${arm_id}_joint1">
+        <hardwareInterface>hardware_interface/EffortJointInterface</hardwareInterface>
+      </joint>
+      <actuator name="${arm_id}_joint1_motor">
+        <hardwareInterface>hardware_interface/EffortJointInterface</hardwareInterface>
+        <mechanicalReduction>1</mechanicalReduction>
+      </actuator>
+    </transmission>
+    <transmission name="${arm_id}_joint2_trans">
+      <type>transmission_interface/SimpleTransmission</type>
+      <joint name="${arm_id}_joint2">
+        <hardwareInterface>hardware_interface/EffortJointInterface</hardwareInterface>
+      </joint>
+      <actuator name="${arm_id}_joint2_motor">
+        <hardwareInterface>hardware_interface/EffortJointInterface</hardwareInterface>
+        <mechanicalReduction>1</mechanicalReduction>
+      </actuator>
+    </transmission>
+    <transmission name="${arm_id}_joint3_trans">
+      <type>transmission_interface/SimpleTransmission</type>
+      <joint name="${arm_id}_joint3">
+        <hardwareInterface>hardware_interface/EffortJointInterface</hardwareInterface>
+      </joint>
+      <actuator name="${arm_id}_joint3_motor">
+        <hardwareInterface>hardware_interface/EffortJointInterface</hardwareInterface>
+        <mechanicalReduction>1</mechanicalReduction>
+      </actuator>
+    </transmission>
+  </xacro:macro>
 </robot>
