Commit message: tried gravity compensation. doesnt seem it works fine.

File: myrobot_description/robots/myrobot.xacro (robot description, xacro)
@@ -11,14 +11,4 @@
     </xacro:unless>
     <xacro:property name="PI" value="3.1415926535897931"/>
-    <xacro:property name="mass" value="1" />
-    <!-- arbitrary value for mass -->
-    <xacro:property name="width" value="0.1" />
-    <!-- Square dimensions (widthxwidth) of beams -->
-    <xacro:property name="height1" value="2" />
-    <!-- Link 1 -->
-    <xacro:property name="height2" value="1" />
-    <!-- Link 2 -->
-    <xacro:property name="height3" value="1" />
-    <!-- Link 3 -->
     <!-- Base Link -->
     <link name="${arm_id}_link1">
@@ -40,6 +30,6 @@
       <inertial>
         <origin xyz="0 0 0" rpy="0 0 0"/>
-        <mass value="${mass}"/>
-        <inertia ixx="${mass / 12.0 * (width*width + height1*height1)}" ixy="0.0" ixz="0.0" iyy="${mass / 12.0 * (height1*height1 + width*width)}" iyz="0.0" izz="${mass / 12.0 * (width*width + width*width)}"/>
+        <mass value="1.0"/>
+        <inertia ixx="1" ixy="0" ixz="1" iyy="0" iyz="1" izz="0"/>
       </inertial>
     </link>
@@ -49,7 +39,6 @@
       <origin xyz="0 0 0.07" rpy="0 0 0"/>
       <axis xyz="0 0 1"/>
-      <dynamics damping="0.7"/>
+      <dynamics damping="0.1"/>
     </joint>
-    <!-- Middle Link -->
     <link name="${arm_id}_link2">
       <collision>
@@ -70,6 +59,6 @@
       <inertial>
         <origin xyz="0 0 0" rpy="0 0 0"/>
-        <mass value="${mass}"/>
-        <inertia ixx="${mass / 12.0 * (width*width + height2*height2)}" ixy="0.0" ixz="0.0" iyy="${mass / 12.0 * (height2*height2 + width*width)}" iyz="0.0" izz="${mass / 12.0 * (width*width + width*width)}"/>
+        <mass value="2.75458"/>
+        <inertia ixx="0.0109697" ixy="-2.08287e-08" ixz="-0.000398309" iyy="0.011856" iyz="2.03974e-09" izz="0.00604953"/>
       </inertial>
     </link>
@@ -79,7 +68,6 @@
       <origin xyz="0.08 0 0.12" rpy="${pi/2} 0 ${pi/2}"/>
       <axis xyz="0 0 1"/>
-      <dynamics damping="0.7"/>
+      <dynamics damping="0.1"/>
     </joint>
-    <!-- Top Link -->
     <link name="${arm_id}_link3">
       <collision>
@@ -100,6 +88,6 @@
       <inertial>
         <origin xyz="0 0 0" rpy="0 0 0"/>
-        <mass value="${mass}"/>
-        <inertia ixx="${mass / 12.0 * (width*width + height3*height3)}" ixy="0.0" ixz="0.0" iyy="${mass / 12.0 * (height3*height3 + width*width)}" iyz="0.0" izz="${mass / 12.0 * (width*width + width*width)}"/>
+        <mass value="8.143"/>
+        <inertia ixx="0.25374" ixy="1.41285e-07" ixz="-7.13886e-08" iyy="0.0212824" iyz="0.00499483" izz="0.247523"/>
       </inertial>
     </link>
@@ -109,7 +97,6 @@
       <origin xyz="0 0.43 0" rpy="0 0 0"/>
       <axis xyz="0 0 1"/>
-      <dynamics damping="0.7"/>
+      <dynamics damping="0.1"/>
     </joint>
-    <!-- Top Link -->
     <link name="${arm_id}_link4">
       <collision>
@@ -130,6 +117,6 @@
       <inertial>
         <origin xyz="0 0 0" rpy="0 0 0"/>
-        <mass value="${mass}"/>
-        <inertia ixx="${mass / 12.0 * (width*width + height3*height3)}" ixy="0.0" ixz="0.0" iyy="${mass / 12.0 * (height3*height3 + width*width)}" iyz="0.0" izz="${mass / 12.0 * (width*width + width*width)}"/>
+        <mass value="5.14886"/>
+        <inertia ixx="0.075434" ixy="2.67415e-08" ixz="2.13561e-09" iyy="0.010425" iyz="0.00274946" izz="0.0744749"/>
       </inertial>
     </link>
